File: MotorController/MotorController.sch (KiCad schematic (older format))
At the start: 15 parts

Commit message: ERC Passed
Connections:
- net GND: now also P?.4 (P4)
- net VCC: now also P?.3 (P3)
Changed lines of the file:
@@
 	3250 4050 3250 4000
 Connection ~ 3050 4050
+$Comp
+L VCC #PWR?
+U 1 1 58EBC3B0
+P 8600 3500
+F 0 "#PWR?" H 8600 3350 50  0001 C CNN
+F 1 "VCC" H 8600 3650 50  0000 C CNN
+F 2 "" H 8600 3500 50  0001 C CNN
+F 3 "" H 8600 3500 50  0001 C CNN
+	1    8600 3500
+	1    0    0    -1
+$EndComp
+$Comp
+L GND #PWR?
+U 1 1 58EBC460
+P 8600 4400
+F 0 "#PWR?" H 8600 4150 50  0001 C CNN
+F 1 "GND" H 8600 4250 50  0000 C CNN
+F 2 "" H 8600 4400 50  0001 C CNN
+F 3 "" H 8600 4400 50  0001 C CNN
+	1    8600 4400
+	1    0    0    -1
+$EndComp
+Wire Wire Line
+	8600 4400 8600 3950
+Wire Wire Line
+	8600 3950 8800 3950
+Wire Wire Line
+	8600 3500 8600 3850
+Wire Wire Line
+	8600 3850 8800 3850
 $EndSCHEMATC

Commit message: Layout terminado sin serigrafia
Parts:
- C1, C2, C3, C4: renamed from C?; footprint (none) -> Capacitors_SMD:C_0805_HandSoldering
- D1: renamed from D?; footprint (none) -> LEDs:LED_0805
- P!1: renamed from P!; footprint (none) -> Connectors_JST:JST_PH_S2B-PH-K_02x2.00mm_Angled
- P1: renamed from P?; footprint (none) -> Connectors_JST:JST_PH_S2B-PH-K_02x2.00mm_Angled
- P2: renamed from P?; footprint (none) -> Pin_Headers:Pin_Header_Straight_1x06_Pitch2.54mm
- R1, R2, R3, R4, R5: renamed from R?; footprint (none) -> Resistors_SMD:R_0805_HandSoldering
- U1, U2: renamed from U?; footprint (none) -> SMD_Packages:SOIC-8-N
Changed lines of the file:
@@
 LIBS:74xgxx
 LIBS:L9110
+LIBS:MotorController-cache
 EELAYER 25 0
 EELAYER END
@@
 $EndDescr
 $Comp
-L L9110 U?
+L L9110 U1
 U 1 1 58EB772B
 P 6150 3400
-F 0 "U?" H 6150 3700 60  0000 C CNN
+F 0 "U1" H 6150 3700 60  0000 C CNN
 F 1 "L9110" H 6150 3100 60  0000 C CNN
-F 2 "" H 6150 3400 60  0000 C CNN
+F 2 "SMD_Packages:SOIC-8-N" H 6150 3400 60  0001 C CNN
 F 3 "" H 6150 3400 60  0000 C CNN
 	1    6150 3400
@@
 $EndComp
 $Comp
-L L9110 U?
+L L9110 U2
 U 1 1 58EB7852
 P 6150 4350
-F 0 "U?" H 6150 4650 60  0000 C CNN
+F 0 "U2" H 6150 4650 60  0000 C CNN
 F 1 "L9110" H 6150 4050 60  0000 C CNN
-F 2 "" H 6150 4350 60  0000 C CNN
+F 2 "SMD_Packages:SOIC-8-N" H 6150 4350 60  0001 C CNN
 F 3 "" H 6150 4350 60  0000 C CNN
 	1    6150 4350
@@
 $EndComp
 $Comp
-L C C?
+L C C3
 U 1 1 58EB7946
 P 5100 3400
-F 0 "C?" H 5125 3500 50  0000 L CNN
+F 0 "C3" H 5125 3500 50  0000 L CNN
 F 1 "0.1uF" H 5125 3300 50  0000 L CNN
-F 2 "" H 5138 3250 50  0001 C CNN
+F 2 "Capacitors_SMD:C_0805_HandSoldering" H 5138 3250 50  0001 C CNN
 F 3 "" H 5100 3400 50  0001 C CNN
 	1    5100 3400
@@
 $EndComp
 $Comp
-L C C?
+L C C4
 U 1 1 58EB79B1
 P 5100 4350
-F 0 "C?" H 5125 4450 50  0000 L CNN
+F 0 "C4" H 5125 4450 50  0000 L CNN
 F 1 "0.1uF" H 5125 4250 50  0000 L CNN
-F 2 "" H 5138 4200 50  0001 C CNN
+F 2 "Capacitors_SMD:C_0805_HandSoldering" H 5138 4200 50  0001 C CNN
 F 3 "" H 5100 4350 50  0001 C CNN
 	1    5100 4350
@@
 $EndComp
 $Comp
-L R R?
+L R R2
 U 1 1 58EB7A1F
 P 7750 2800
-F 0 "R?" V 7830 2800 50  0000 C CNN
+F 0 "R2" V 7830 2800 50  0000 C CNN
 F 1 "10K" V 7750 2800 50  0000 C CNN
-F 2 "" V 7680 2800 50  0001 C CNN
+F 2 "Resistors_SMD:R_0805_HandSoldering" V 7680 2800 50  0001 C CNN
 F 3 "" H 7750 2800 50  0001 C CNN
 	1    7750 2800
@@
 $EndComp
 $Comp
-L LED D?
+L LED D1
 U 1 1 58EB7A74
 P 4000 4000
-F 0 "D?" H 4000 4100 50  0000 C CNN
+F 0 "D1" H 4000 4100 50  0000 C CNN
 F 1 "LED" H 4000 3900 50  0000 C CNN
-F 2 "" H 4000 4000 50  0001 C CNN
+F 2 "LEDs:LED_0805" H 4000 4000 50  0001 C CNN
 F 3 "" H 4000 4000 50  0001 C CNN
 	1    4000 4000
@@
 $EndComp
 $Comp
-L VCC #PWR?
+L VCC #PWR01
 U 1 1 58EB7AD9
 P 5400 2950
-F 0 "#PWR?" H 5400 2800 50  0001 C CNN
+F 0 "#PWR01" H 5400 2800 50  0001 C CNN
 F 1 "VCC" H 5400 3100 50  0000 C CNN
 F 2 "" H 5400 2950 50  0001 C CNN
@@
 $EndComp
 $Comp
-L GND #PWR?
+L GND #PWR02
 U 1 1 58EB7AF9
 P 6900 4800
-F 0 "#PWR?" H 6900 4550 50  0001 C CNN
+F 0 "#PWR02" H 6900 4550 50  0001 C CNN
 F 1 "GND" H 6900 4650 50  0000 C CNN
 F 2 "" H 6900 4800 50  0001 C CNN
@@
 $EndComp
 $Comp
-L CONN_01X06 P?
+L CONN_01X06 P2
 U 1 1 58EB7E0D
 P 9000 3900
-F 0 "P?" H 9000 4250 50  0000 C CNN
+F 0 "P2" H 9000 4250 50  0000 C CNN
 F 1 "CONN_01X06" V 9100 3900 50  0000 C CNN
-F 2 "" H 9000 3900 50  0001 C CNN
+F 2 "Pin_Headers:Pin_Header_Straight_1x06_Pitch2.54mm" H 9000 3900 50  0001 C CNN
 F 3 "" H 9000 3900 50  0001 C CNN
 	1    9000 3900
@@
 $EndComp
 $Comp
-L CONN_01X02 P!
+L CONN_01X02 P!1
 U 1 1 58EB7E66
 P 4450 3400
-F 0 "P!" H 4450 3550 50  0000 C CNN
+F 0 "P!1" H 4450 3550 50  0000 C CNN
 F 1 "MOTOR_1" V 4550 3400 50  0000 C CNN
-F 2 "" H 4450 3400 50  0001 C CNN
+F 2 "Connectors_JST:JST_PH_S2B-PH-K_02x2.00mm_Angled" H 4450 3400 50  0001 C CNN
 F 3 "" H 4450 3400 50  0001 C CNN
 	1    4450 3400
@@
 $EndComp
 $Comp
-L CONN_01X02 P?
+L CONN_01X02 P1
 U 1 1 58EB7EFB
 P 4450 4350
-F 0 "P?" H 4450 4500 50  0000 C CNN
+F 0 "P1" H 4450 4500 50  0000 C CNN
 F 1 "MOTOR_2" V 4550 4350 50  0000 C CNN
-F 2 "" H 4450 4350 50  0001 C CNN
+F 2 "Connectors_JST:JST_PH_S2B-PH-K_02x2.00mm_Angled" H 4450 4350 50  0001 C CNN
 F 3 "" H 4450 4350 50  0001 C CNN
 	1    4450 4350
@@
 $EndComp
 $Comp
-L R R?
+L R R3
 U 1 1 58EB9964
 P 7950 2800
-F 0 "R?" V 8030 2800 50  0000 C CNN
+F 0 "R3" V 8030 2800 50  0000 C CNN
 F 1 "10K" V 7950 2800 50  0000 C CNN
-F 2 "" V 7880 2800 50  0001 C CNN
+F 2 "Resistors_SMD:R_0805_HandSoldering" V 7880 2800 50  0001 C CNN
 F 3 "" H 7950 2800 50  0001 C CNN
 	1    7950 2800
@@
 $EndComp
 $Comp
-L R R?
+L R R4
 U 1 1 58EB9996
 P 8150 2800
-F 0 "R?" V 8230 2800 50  0000 C CNN
+F 0 "R4" V 8230 2800 50  0000 C CNN
 F 1 "10K" V 8150 2800 50  0000 C CNN
-F 2 "" V 8080 2800 50  0001 C CNN
+F 2 "Resistors_SMD:R_0805_HandSoldering" V 8080 2800 50  0001 C CNN
 F 3 "" H 8150 2800 50  0001 C CNN
 	1    8150 2800
@@
 $EndComp
 $Comp
-L R R?
+L R R5
 U 1 1 58EB99CB
 P 8350 2800
-F 0 "R?" V 8430 2800 50  0000 C CNN
+F 0 "R5" V 8430 2800 50  0000 C CNN
 F 1 "10K" V 8350 2800 50  0000 C CNN
-F 2 "" V 8280 2800 50  0001 C CNN
+F 2 "Resistors_SMD:R_0805_HandSoldering" V 8280 2800 50  0001 C CNN
 F 3 "" H 8350 2800 50  0001 C CNN
 	1    8350 2800
@@
 Connection ~ 8350 4150
 $Comp
-L VCC #PWR?
+L VCC #PWR03
 U 1 1 58EBA40F
 P 8050 2400
-F 0 "#PWR?" H 8050 2250 50  0001 C CNN
+F 0 "#PWR03" H 8050 2250 50  0001 C CNN
 F 1 "VCC" H 8050 2550 50  0000 C CNN
 F 2 "" H 8050 2400 50  0001 C CNN
@@
 Connection ~ 8150 2500
 $Comp
-L VCC #PWR?
+L VCC #PWR04
 U 1 1 58EBA735
 P 4000 3450
-F 0 "#PWR?" H 4000 3300 50  0001 C CNN
+F 0 "#PWR04" H 4000 3300 50  0001 C CNN
 F 1 "VCC" H 4000 3600 50  0000 C CNN
 F 2 "" H 4000 3450 50  0001 C CNN
@@
 $EndComp
 $Comp
-L R R?
+L R R1
 U 1 1 58EBA8D6
 P 4000 3650
-F 0 "R?" V 4080 3650 50  0000 C CNN
+F 0 "R1" V 4080 3650 50  0000 C CNN
 F 1 "1K" V 4000 3650 50  0000 C CNN
-F 2 "" V 3930 3650 50  0001 C CNN
+F 2 "Resistors_SMD:R_0805_HandSoldering" V 3930 3650 50  0001 C CNN
 F 3 "" H 4000 3650 50  0001 C CNN
 	1    4000 3650
@@
 	4000 3800 4000 3850
 $Comp
-L GND #PWR?
+L GND #PWR05
 U 1 1 58EBAC5F
 P 4000 4250
-F 0 "#PWR?" H 4000 4000 50  0001 C CNN
+F 0 "#PWR05" H 4000 4000 50  0001 C CNN
 F 1 "GND" H 4000 4100 50  0000 C CNN
 F 2 "" H 4000 4250 50  0001 C CNN
@@
 	4000 4150 4000 4250
 $Comp
-L C C?
+L C C1
 U 1 1 58EBB1AD
 P 2850 3850
-F 0 "C?" H 2875 3950 50  0000 L CNN
+F 0 "C1" H 2875 3950 50  0000 L CNN
 F 1 "10uF" H 2875 3750 50  0000 L CNN
-F 2 "" H 2888 3700 50  0001 C CNN
+F 2 "Capacitors_SMD:C_0805_HandSoldering" H 2888 3700 50  0001 C CNN
 F 3 "" H 2850 3850 50  0001 C CNN
 	1    2850 3850
@@
 $EndComp
 $Comp
-L C C?
+L C C2
 U 1 1 58EBB323
 P 3250 3850
-F 0 "C?" H 3275 3950 50  0000 L CNN
+F 0 "C2" H 3275 3950 50  0000 L CNN
 F 1 "0.1uF" H 3275 3750 50  0000 L CNN
-F 2 "" H 3288 3700 50  0001 C CNN
+F 2 "Capacitors_SMD:C_0805_HandSoldering" H 3288 3700 50  0001 C CNN
 F 3 "" H 3250 3850 50  0001 C CNN
 	1    3250 3850
@@
 $EndComp
 $Comp
-L VCC #PWR?
+L VCC #PWR06
 U 1 1 58EBB408
 P 3050 3600
-F 0 "#PWR?" H 3050 3450 50  0001 C CNN
+F 0 "#PWR06" H 3050 3450 50  0001 C CNN
 F 1 "VCC" H 3050 3750 50  0000 C CNN
 F 2 "" H 3050 3600 50  0001 C CNN
@@
 $EndComp
 $Comp
-L GND #PWR?
+L GND #PWR07
 U 1 1 58EBB6A6
 P 3050 4100
-F 0 "#PWR?" H 3050 3850 50  0001 C CNN
+F 0 "#PWR07" H 3050 3850 50  0001 C CNN
 F 1 "GND" H 3050 3950 50  0000 C CNN
 F 2 "" H 3050 4100 50  0001 C CNN
@@
 Connection ~ 3050 4050
 $Comp
-L VCC #PWR?
+L VCC #PWR08
 U 1 1 58EBC3B0
 P 8600 3500
-F 0 "#PWR?" H 8600 3350 50  0001 C CNN
+F 0 "#PWR08" H 8600 3350 50  0001 C CNN
 F 1 "VCC" H 8600 3650 50  0000 C CNN
 F 2 "" H 8600 3500 50  0001 C CNN
@@
 $EndComp
 $Comp
-L GND #PWR?
+L GND #PWR09
 U 1 1 58EBC460
 P 8600 4400
-F 0 "#PWR?" H 8600 4150 50  0001 C CNN
+F 0 "#PWR09" H 8600 4150 50  0001 C CNN
 F 1 "GND" H 8600 4250 50  0000 C CNN
 F 2 "" H 8600 4400 50  0001 C CNN
@@
 Wire Wire Line
 	8600 3850 8800 3850
+$Comp
+L PWR_FLAG #FLG010
+U 1 1 58EBD6F1
+P 6200 6700
+F 0 "#FLG010" H 6200 6775 50  0001 C CNN
+F 1 "PWR_FLAG" H 6200 6850 50  0000 C CNN
+F 2 "" H 6200 6700 50  0001 C CNN
+F 3 "" H 6200 6700 50  0001 C CNN
+	1    6200 6700
+	1    0    0    -1
+$EndComp
+$Comp
+L GND #PWR011
+U 1 1 58EBD799
+P 6200 6950
+F 0 "#PWR011" H 6200 6700 50  0001 C CNN
+F 1 "GND" H 6200 6800 50  0000 C CNN
+F 2 "" H 6200 6950 50  0001 C CNN
+F 3 "" H 6200 6950 50  0001 C CNN
+	1    6200 6950
+	1    0    0    -1
+$EndComp
+Wire Wire Line
+	6200 6700 6200 6950
+$Comp
+L PWR_FLAG #FLG012
+U 1 1 58EBD89B
+P 6600 6950
+F 0 "#FLG012" H 6600 7025 50  0001 C CNN
+F 1 "PWR_FLAG" H 6600 7100 50  0000 C CNN
+F 2 "" H 6600 6950 50  0001 C CNN
+F 3 "" H 6600 6950 50  0001 C CNN
+	1    6600 6950
+	-1   0    0    1
+$EndComp
+$Comp
+L VCC #PWR013
+U 1 1 58EBD9D9
+P 6600 6700
+F 0 "#PWR013" H 6600 6550 50  0001 C CNN
+F 1 "VCC" H 6600 6850 50  0000 C CNN
+F 2 "" H 6600 6700 50  0001 C CNN
+F 3 "" H 6600 6700 50  0001 C CNN
+	1    6600 6700
+	1    0    0    -1
+$EndComp
+Wire Wire Line
+	6600 6700 6600 6950
 $EndSCHEMATC
